Commit message: feat:完成底盘可通过cmd_vel控制

File: src/chassis_description/urdf/chassis.urdf.xacro (robot description, xacro)
@@ -219,4 +219,8 @@
       name="gz_ros2_control::GazeboSimROS2ControlPlugin">
       <parameters>$(find chassis_description)/config/ros2_controllers.yaml</parameters>
+      <ros>
+        <remapping>cmd_vel:=/cmd_vel</remapping>
+        <remapping>odom:=/odom</remapping>
+      </ros>
     </plugin>
   </gazebo>

File: src/chassis_description/urdf/macros.xacro (robot description, xacro)
@@ -55,5 +55,5 @@
       <!-- 支撑臂（简化成一根斜臂） -->
       <visual>
-        <origin xyz="0 0 -${wheel_center_drop/2.0}" rpy="0.35 0 0"/>
+        <origin xyz="0 0 -${wheel_center_drop/2.0}" rpy="0 0 0"/>
         <geometry>
           <box size="${arm_thickness} ${wheel_width*0.9} ${arm_length}"/>
